File: badge-kicad.sch (KiCad schematic (older format))
At the start: 112 parts, among them J2 JTAG, P2 CONN_02X20, P3 FTDI BACKUP, P4 USB_MICRO_RIGHT, P5 LED OUT (DNP), SW1 RESET, SW2 POWERON, SW3 TM1000, SW4 UP, SW5 DN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

Commit message: fix typo
Other:
- note added: "rev1 did not connect VR_PA and its cap/inductor pair\n"
- note removed: "rev1 did not connect VR_PA and it’s cap/inductor pair\n"
Changed lines of the file:
@@
 VR_PA
 Text Notes 7050 5400 0    60   ~ 0
-rev1 did not connect VR_PA and it’s cap/inductor pair\n
+rev1 did not connect VR_PA and its cap/inductor pair\n
 $Comp
 L GND #PWR038

Commit message: update for fabrication rev3
Parts:
- added TP11: PTC1, Measurement_Points:Measurement_Point_Round-TH_Small, symbol TEST
- added TP12: PTB0, Measurement_Points:Measurement_Point_Round-TH_Small, symbol TEST
- added TP13: PTE16, Measurement_Points:Measurement_Point_Round-TH_Small, symbol TEST
- added TP14: PTB1, Measurement_Points:Measurement_Point_Round-TH_Small, symbol TEST
- added TP6: PTA19, Measurement_Points:Measurement_Point_Round-TH_Small, symbol TEST
- added TP7: PTC2, Measurement_Points:Measurement_Point_Round-TH_Small, symbol TEST
- added TP8: PTC4, Measurement_Points:Measurement_Point_Round-TH_Small, symbol TEST
- BT1: value Battery 3.7v 1000mAh -> Battery 3.7v 1200mAh
Connections:
- net PTB0: now also TP12.1
- net PTB1: now also TP14.1
- net PTE16: now also TP13.1
- net SWDN: now also TP8.1
- net SWL: now also TP7.1
- net SWR: now also TP11.1
- net SWUP: now also TP6.1
- net VBAT: now also SW2.2 (NC); no longer BT1.1, C15.1, U16.3 (VBAT)
- net VCC: now also U15.5 (VOUT); no longer SW2.2 (NC)
- net VCHG: now reaches SW2.1 (COM)
- net VCHG: now also BT1.1, C15.1, U16.3 (VBAT); no longer U15.5 (VOUT)
Other:
- moved on the sheet: SW2
Changed lines of the file:
@@
 P 4000 1400
 F 0 "BT1" V 4150 1300 50  0000 L CNN
-F 1 "Battery 3.7v 1000mAh" V 4300 750 50  0000 L CNN
+F 1 "Battery 3.7v 1200mAh" V 3850 1050 50  0000 L CNN
 F 2 "Connectors_JST:JST_PH_S2B-PH-SM4-TB_02x2.00mm_Angled" V 4000 1440 50  0001 C CNN
 F 3 "" V 4000 1440 50  0000 C CNN
@@
 Text GLabel 3050 4300 1    60   Input ~ 0
 RF_RESET
-Text Notes 3900 650  0    60   ~ 12
+Text Notes 3850 600  0    60   ~ 12
 Power / Charge
 Text GLabel 14500 6600 0    60   Input ~ 0
@@
 	1    0    0    -1
 $EndComp
-Text GLabel 4150 850  0    60   Input ~ 0
+Text GLabel 4000 950  1    60   Input ~ 0
 VCHG
 $Comp
@@
 P 4700 1000
 F 0 "#FLG031" H 4700 1095 50  0001 C CNN
-F 1 "PWR_FLAG" H 4700 1224 50  0000 C CNN
+F 1 "PWR_FLAG" H 4950 1100 50  0000 C CNN
 F 2 "" H 4700 1000 50  0000 C CNN
 F 3 "" H 4700 1000 50  0000 C CNN
@@
 Text GLabel 12100 1900 1    60   Input ~ 0
 VBAT
-Text GLabel 4350 950  1    60   Output ~ 0
+Text GLabel 4500 900  1    60   Output ~ 0
 VBAT
 Text Notes 12150 1600 0    60   ~ 0
@@
 Text GLabel 6450 8150 2    60   Output ~ 0
 RF_RESET
-Text Notes 15500 8950 0    60   ~ 0
+Text Notes 15750 8950 0    60   ~ 0
 Radio RX
-Text Notes 15500 8600 0    60   ~ 0
+Text Notes 15750 8600 0    60   ~ 0
 Radio TX
-Text Notes 15500 8200 0    60   ~ 0
+Text Notes 15750 8200 0    60   ~ 0
 SD Card I/O\n
 $Comp
@@
 L SW_SPDT SW2
 U 1 1 585C7C26
-P 5950 1100
-F 0 "SW2" H 6000 1400 50  0000 C CNN
-F 1 "POWERON" H 6000 1300 50  0000 C CNN
-F 2 "Buttons_Switches_SMD:SW_SPDT_PCM12" H 5950 1100 60  0001 C CNN
-F 3 "" H 5950 1100 60  0000 C CNN
-	1    5950 1100
-	1    0    0    -1
-$EndComp
-NoConn ~ 6100 1150
+P 4250 1150
+F 0 "SW2" H 4300 1450 50  0000 C CNN
+F 1 "POWERON" H 4300 1350 50  0000 C CNN
+F 2 "Buttons_Switches_SMD:SW_SPDT_PCM12" H 4250 1150 60  0001 C CNN
+F 3 "" H 4250 1150 60  0000 C CNN
+	1    4250 1150
+	1    0    0    -1
+$EndComp
 $Comp
 L USB_MICRO_RIGHT P4
@@
 $Comp
 L PWR_FLAG #FLG036
-U 1 1 585EF217
-P 6550 900
-F 0 "#FLG036" H 6550 995 50  0001 C CNN
-F 1 "PWR_FLAG" H 6550 1124 50  0000 C CNN
-F 2 "" H 6550 900 50  0000 C CNN
-F 3 "" H 6550 900 50  0000 C CNN
-	1    6550 900
-	1    0    0    -1
-$EndComp
-$Comp
-L PWR_FLAG #FLG037
 U 1 1 585EF776
 P 8050 7900
-F 0 "#FLG037" H 8050 7995 50  0001 C CNN
+F 0 "#FLG036" H 8050 7995 50  0001 C CNN
 F 1 "PWR_FLAG" H 7750 8000 50  0000 C CNN
 F 2 "" H 8050 7900 50  0000 C CNN
@@
 rev1 did not connect VR_PA and its cap/inductor pair\n
 $Comp
-L GND #PWR038
+L GND #PWR037
 U 1 1 58606D55
 P 9150 7450
-F 0 "#PWR038" H 9150 7200 50  0001 C CNN
+F 0 "#PWR037" H 9150 7200 50  0001 C CNN
 F 1 "GND" H 9155 7277 50  0000 C CNN
 F 2 "" H 9150 7450 50  0000 C CNN
@@
 $EndComp
 $Comp
-L GND #PWR039
+L GND #PWR038
 U 1 1 586304A7
 P 7250 6050
-F 0 "#PWR039" H 7250 5800 50  0001 C CNN
+F 0 "#PWR038" H 7250 5800 50  0001 C CNN
 F 1 "GND" H 7255 5877 50  0000 C CNN
 F 2 "" H 7250 6050 50  0000 C CNN
@@
 	0    -1   1    0
 $EndComp
-Text Notes 14650 1900 0    60   ~ 0
+Text Notes 14550 1650 0    60   ~ 0
 Extra Test Pins\n
 $Comp
@@
 $EndComp
 $Comp
-L GND #PWR040
+L GND #PWR039
 U 1 1 588B02C8
 P 16400 2950
-F 0 "#PWR040" H 16400 2700 50  0001 C CNN
+F 0 "#PWR039" H 16400 2700 50  0001 C CNN
 F 1 "GND" H 16405 2777 50  0000 C CNN
 F 2 "" H 16400 2950 50  0000 C CNN
@@
 $EndComp
 $Comp
-L VCC #PWR041
+L VCC #PWR040
 U 1 1 588B394B
 P 16300 1900
-F 0 "#PWR041" H 16300 1750 50  0001 C CNN
+F 0 "#PWR040" H 16300 1750 50  0001 C CNN
 F 1 "VCC" H 16317 2073 50  0000 C CNN
 F 2 "" H 16300 1900 50  0000 C CNN
@@
 $EndComp
 $Comp
-L GND #PWR042
+L GND #PWR041
 U 1 1 588DEEDE
 P 3450 4000
-F 0 "#PWR042" H 3450 3750 50  0001 C CNN
+F 0 "#PWR041" H 3450 3750 50  0001 C CNN
 F 1 "GND" H 3350 4000 50  0000 C CNN
 F 2 "" H 3450 4000 50  0000 C CNN
@@
 $EndComp
 $Comp
-L GND #PWR043
+L GND #PWR042
 U 1 1 588DF442
 P 3700 3500
-F 0 "#PWR043" H 3700 3250 50  0001 C CNN
+F 0 "#PWR042" H 3700 3250 50  0001 C CNN
 F 1 "GND" H 3600 3500 50  0000 C CNN
 F 2 "" H 3700 3500 50  0000 C CNN
@@
 $EndComp
 $Comp
-L GND #PWR044
+L GND #PWR043
 U 1 1 588E38CC
 P 2200 4100
-F 0 "#PWR044" H 2200 3850 50  0001 C CNN
+F 0 "#PWR043" H 2200 3850 50  0001 C CNN
 F 1 "GND" H 2205 3927 50  0000 C CNN
 F 2 "" H 2200 4100 50  0000 C CNN
@@
 $EndComp
 $Comp
-L GND #PWR045
+L GND #PWR044
 U 1 1 588E4DB4
 P 4600 4050
-F 0 "#PWR045" H 4600 3800 50  0001 C CNN
+F 0 "#PWR044" H 4600 3800 50  0001 C CNN
 F 1 "GND" H 4605 3877 50  0000 C CNN
 F 2 "" H 4600 4050 50  0000 C CNN
@@
 $EndComp
 $Comp
-L GND #PWR046
+L GND #PWR045
 U 1 1 588EB7C8
 P 7100 10300
-F 0 "#PWR046" H 7100 10050 50  0001 C CNN
+F 0 "#PWR045" H 7100 10050 50  0001 C CNN
 F 1 "GND" H 7105 10127 50  0000 C CNN
 F 2 "" H 7100 10300 50  0000 C CNN
@@
 Text GLabel 1550 6950 0    60   Input ~ 0
 SWENTER
-Text GLabel 2100 9650 0    60   Input ~ 0
+Text GLabel 1150 9650 0    60   Input ~ 0
 SWUP
 Text GLabel 4300 10000 2    60   Input ~ 0
 SWDN
-Text GLabel 3500 10000 3    60   Input ~ 0
+Text GLabel 3500 10200 3    60   Input ~ 0
 SWL
 Text GLabel 4300 10300 2    60   Input ~ 0
@@
 $EndComp
 $Comp
-L GND #PWR047
+L GND #PWR046
 U 1 1 589B031F
 P 6650 7250
-F 0 "#PWR047" H 6650 7000 50  0001 C CNN
+F 0 "#PWR046" H 6650 7000 50  0001 C CNN
 F 1 "GND" H 6800 7250 50  0000 C CNN
 F 2 "" H 6650 7250 50  0000 C CNN
@@
 	1700 6100 1850 6100
 Wire Wire Line
-	3500 9200 3500 10000
+	3500 9200 3500 10200
 Wire Wire Line
 	2900 4700 2900 4900
@@
 	4000 1550 4000 1700
 Wire Wire Line
-	4000 1100 4000 1250
+	4000 950  4000 1250
 Wire Wire Line
 	4550 1100 4550 1300
@@
 	4500 1600 4500 1650
 Wire Wire Line
-	4500 1100 4500 1300
-Wire Wire Line
-	4150 850  4200 850
-Wire Wire Line
-	4200 850  4200 1100
-Connection ~ 4200 1100
+	4500 900  4500 1300
 Wire Wire Line
 	6800 3000 6800 3200
@@
 Connection ~ 5200 2500
 Wire Wire Line
-	4000 1100 4800 1100
-Wire Wire Line
 	4700 1000 4700 1100
 Connection ~ 4700 1100
-Wire Wire Line
-	4350 950  4350 1100
-Connection ~ 4350 1100
 Wire Wire Line
 	8500 2800 8700 2800
@@
 	13850 8050 13850 8150
 Wire Wire Line
-	5600 1100 5800 1100
+	5600 1100 6100 1100
 Wire Wire Line
 	6100 1050 6800 1050
@@
 	13400 1900 13400 2400
 Connection ~ 13400 2400
-Wire Wire Line
-	6550 900  6550 1050
-Connection ~ 6550 1050
 Connection ~ 8050 8350
 Wire Wire Line
@@
 Connection ~ 3800 9400
 Wire Wire Line
-	2100 9650 2500 9650
+	1150 9650 2500 9650
 Connection ~ 2500 9650
 Wire Notes Line
@@
 Connection ~ 2600 4700
 $Comp
-L GND #PWR?
+L GND #PWR047
 U 1 1 589B5800
 P 2250 4900
-F 0 "#PWR?" H 2250 4650 50  0001 C CNN
+F 0 "#PWR047" H 2250 4650 50  0001 C CNN
 F 1 "GND" H 2250 4750 50  0000 C CNN
 F 2 "" H 2250 4900 50  0000 C CNN
@@
 	1    0    0    -1
 $EndComp
+$Comp
+L TEST TP8
+U 1 1 58B4CB31
+P 4200 9800
+F 0 "TP8" H 4278 9940 50  0000 L CNN
+F 1 "PTC4" H 4278 9849 50  0000 L CNN
+F 2 "Measurement_Points:Measurement_Point_Round-TH_Small" H 4200 9800 50  0001 C CNN
+F 3 "" H 4200 9800 50  0000 C CNN
+	1    4200 9800
+	1    0    0    -1
+$EndComp
+Wire Wire Line
+	4200 9800 4200 10000
+Connection ~ 4200 10000
+$Comp
+L TEST TP11
+U 1 1 58B4D07C
+P 4900 10150
+F 0 "TP11" H 4978 10290 50  0000 L CNN
+F 1 "PTC1" H 4978 10199 50  0000 L CNN
+F 2 "Measurement_Points:Measurement_Point_Round-TH_Small" H 4900 10150 50  0001 C CNN
+F 3 "" H 4900 10150 50  0000 C CNN
+	1    4900 10150
+	1    0    0    -1
+$EndComp
+Wire Wire Line
+	4150 10300 4150 10150
+Wire Wire Line
+	4150 10150 4900 10150
+Connection ~ 4150 10300
+$Comp
+L TEST TP7
+U 1 1 58B4D5BD
+P 3200 9850
+F 0 "TP7" H 3278 9990 50  0000 L CNN
+F 1 "PTC2" H 3278 9899 50  0000 L CNN
+F 2 "Measurement_Points:Measurement_Point_Round-TH_Small" H 3200 9850 50  0001 C CNN
+F 3 "" H 3200 9850 50  0000 C CNN
+	1    3200 9850
+	1    0    0    -1
+$EndComp
+Wire Wire Line
+	3200 9850 3200 9950
+Wire Wire Line
+	3200 9950 3500 9950
+Connection ~ 3500 9950
+$Comp
+L TEST TP6
+U 1 1 58B4E5CE
+P 1250 9450
+F 0 "TP6" H 1328 9590 50  0000 L CNN
+F 1 "PTA19" H 1328 9499 50  0000 L CNN
+F 2 "Measurement_Points:Measurement_Point_Round-TH_Small" H 1250 9450 50  0001 C CNN
+F 3 "" H 1250 9450 50  0000 C CNN
+	1    1250 9450
+	1    0    0    -1
+$EndComp
+Wire Wire Line
+	1250 9450 1250 9650
+Connection ~ 1250 9650
+$Comp
+L TEST TP12
+U 1 1 58B53949
+P 15300 7900
+F 0 "TP12" H 15378 8040 50  0000 L CNN
+F 1 "PTB0" H 15378 7949 50  0000 L CNN
+F 2 "Measurement_Points:Measurement_Point_Round-TH_Small" H 15300 7900 50  0001 C CNN
+F 3 "" H 15300 7900 50  0000 C CNN
+	1    15300 7900
+	1    0    0    -1
+$EndComp
+Wire Wire Line
+	15300 7900 15300 8050
+Connection ~ 15300 8050
+$Comp
+L TEST TP13
+U 1 1 58B5419C
+P 15300 8350
+F 0 "TP13" H 15378 8490 50  0000 L CNN
+F 1 "PTE16" H 15378 8399 50  0000 L CNN
+F 2 "Measurement_Points:Measurement_Point_Round-TH_Small" H 15300 8350 50  0001 C CNN
+F 3 "" H 15300 8350 50  0000 C CNN
+	1    15300 8350
+	1    0    0    -1
+$EndComp
+Wire Wire Line
+	15300 8350 15300 8450
+Connection ~ 15300 8450
+$Comp
+L TEST TP14
+U 1 1 58B54606
+P 15400 9000
+F 0 "TP14" H 15150 9100 50  0000 L CNN
+F 1 "PTB1" H 15100 9200 50  0000 L CNN
+F 2 "Measurement_Points:Measurement_Point_Round-TH_Small" H 15400 9000 50  0001 C CNN
+F 3 "" H 15400 9000 50  0000 C CNN
+	1    15400 9000
+	-1   0    0    1
+$EndComp
+Wire Wire Line
+	15400 9000 15400 8800
+Connection ~ 15400 8800
+Wire Wire Line
+	6100 1100 6100 1050
+Wire Wire Line
+	4100 1150 4000 1150
+Connection ~ 4000 1150
+Wire Wire Line
+	4400 1100 4800 1100
+NoConn ~ 4400 1200
 $EndSCHEMATC
