File: badge_audio.sch (KiCad schematic (older format))
At the start: 15 parts, among them U18 LM386

Commit message: Final rev2, clean up rev1
Parts:
- C44: footprint Capacitors_SMD:C_0805_HandSoldering -> Capacitors_SMD:C_0603_HandSoldering
Changed lines of the file:
@@
 	4100 4050 3900 4050
 $Comp
-L GND #PWR053
+L GND #PWR047
 U 1 1 5894DD97
 P 6050 4400
-F 0 "#PWR053" H 6050 4150 50  0001 C CNN
+F 0 "#PWR047" H 6050 4150 50  0001 C CNN
 F 1 "GND" H 6055 4227 50  0000 C CNN
 F 2 "" H 6050 4400 50  0000 C CNN
@@
 	6700 3100 6700 3550
 $Comp
-L GND #PWR054
+L GND #PWR048
 U 1 1 5894DDAA
 P 6950 3500
-F 0 "#PWR054" H 6950 3250 50  0001 C CNN
+F 0 "#PWR048" H 6950 3250 50  0001 C CNN
 F 1 "GND" H 6955 3327 50  0000 C CNN
 F 2 "" H 6950 3500 50  0000 C CNN
@@
 F 0 "C44" H 5350 4150 50  0000 L CNN
 F 1 "0.01uF" H 5250 4050 50  0000 L CNN
-F 2 "Capacitors_SMD:C_0805_HandSoldering" H 5688 3950 50  0001 C CNN
+F 2 "Capacitors_SMD:C_0603_HandSoldering" H 5688 3950 50  0001 C CNN
 F 3 "" H 5650 4100 50  0000 C CNN
 	1    5650 4100
@@
 $EndComp
 $Comp
-L GND #PWR055
+L GND #PWR049
 U 1 1 5894DDFD
 P 7250 4950
-F 0 "#PWR055" H 7250 4700 50  0001 C CNN
+F 0 "#PWR049" H 7250 4700 50  0001 C CNN
 F 1 "GND" H 7255 4777 50  0000 C CNN
 F 2 "" H 7250 4950 50  0000 C CNN
@@
 $EndComp
 $Comp
-L GND #PWR056
+L GND #PWR050
 U 1 1 58945FCC
 P 6100 3400
-F 0 "#PWR056" H 6100 3150 50  0001 C CNN
+F 0 "#PWR050" H 6100 3150 50  0001 C CNN
 F 1 "GND" H 6100 3250 50  0000 C CNN
 F 2 "" H 6100 3400 50  0000 C CNN

Commit message: update for fabrication rev3
Parts:
- SP2: value MODEL TBD -> AST_01708MR_R
Changed lines of the file:
@@
 P 8200 3950
 F 0 "SP2" H 8200 4300 50  0000 C CNN
-F 1 "MODEL TBD" H 8250 3550 50  0000 C CNN
+F 1 "AST_01708MR_R" H 8250 3550 50  0000 C CNN
 F 2 "jna-parts:SPEAKER_AST_01708MR_R" H 8200 3950 50  0001 C CNN
 F 3 "" H 8200 3950 50  0000 C CNN
