File: fabrication-rev3/badge-kicad.kicad_pcb (KiCad board)
At the start: 2 copper layers, 152.7 x 76.7 mm, 139 parts, among them J2 JTAG, P2 CONN_02X20, P3 FTDI BACKUP, P4 USB_MICRO_RIGHT, P5 LED OUT (DNP), SW1 RESET, SW2 POWERON, SW3 TM1000, SW4 UP, SW5 DN, SW6 LEFT, SW7 RIGHT, SW8 ENTER, U1 WS2812B, U10 WS2812B, U11 WS2812B, U12 WS2812B, U13 MKW01Z128, U14 FT232RL SSOP, U15 MF-REG-SOT235-3.3V-300mA, U16 MCP73831T-2ACI/OT, U18 LM386, U2 WS2812B, U3 WS2812B, U4 WS2812B, U5 WS2812B, U6 WS2812B, U7 WS2812B, U8 WS2812B, U9 WS2812B, Y1 EXS00A-CS02368

Commit message: check in changes before modifiying footprint for rev4
Parts:
- added G***: LOGO, logos:avast_36_11, B.Cu at (161.6, 62.0)
- P4: value USB_MICRO_RIGHT -> CHARGE/CONSOLE
- moved ? 49.2 mm to (132.9, 118.4)
- moved ? 15.0 mm to (166.2, 121.1)
- moved C43 11.1 mm to (166.2, 77.2), turned to 270 degrees
- moved R19 6.40 mm to (163.2, 81.7), turned to 270 degrees
- moved ? 4.93 mm to (164.8, 74.1)
- moved C47 4.09 mm to (170.3, 85.2), turned to 270 degrees
- moved C36 3.22 mm to (143.2, 80.8), turned to 180 degrees
- moved C25 2.55 mm to (125.4, 66.8)
- moved C34 1.24 mm to (139.8, 84.9), turned to 90 degrees
- moved C42 1.21 mm to (163.2, 77.2), turned to 270 degrees
- moved R20 0.73 mm to (166.3, 81.7), turned to 270 degrees
- moved R22 0.60 mm to (166.2, 72.7), turned to 90 degrees
Routing:
- net GND: track 762.3 -> 715.1 mm
- net Net-(C42-Pad1): track 34.7 -> 15.4 mm
- net Net-(C43-Pad2): track 21.0 -> 2.27 mm
- net Net-(C26-Pad1): track 46.1 -> 31.7 mm
- net PWM_SOUND: track 32.7 -> 23.8 mm
- net VCC: track 321.3 -> 328.6 mm, vias 9 -> 8
- net PTB0: track 130.9 -> 136.6 mm
- net Net-(C47-Pad1): track 42.9 -> 37.6 mm
- net Net-(C42-Pad2): track 5.07 -> 2.36 mm
- net Net-(C47-Pad2): track 9.01 -> 6.62 mm
- net Net-(C25-Pad1): track 8.79 -> 6.76 mm
- net CLOCKOUT: track 43.2 -> 41.5 mm
- net DACOUT: track 60.1 -> 58.7 mm
- net UART_RX: track 54.5 -> 55.7 mm
- net Net-(C44-Pad1): track 29.2 -> 30.2 mm
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Other:
- board text added: "CHARGED"
- board text added: "VBATT (+)"
- board text removed: "CHG DONE"
